Commit message: 导航收敛：nav2/localization 参数调优、nav.launch 重构、底盘与里程计微调

File: ros2_ws/src/armbot_description/urdf/armbot.urdf.xacro (robot description, xacro)
@@ -56,5 +56,5 @@
     <parent link="base_link"/>
     <child link="base_lidar_link"/>
-    <origin xyz="0 0 0.15" rpy="0 0 0"/>
+    <origin xyz="0.175 0 0.15" rpy="0 0 0"/>
   </joint>
   <link name="base_lidar_link">
