Commit message: fix: 雷达 0° 朝车尾装反，laser tf yaw 补偿 180°（URDF/nav.launch）

File: ros2_ws/src/armbot_description/urdf/armbot.urdf.xacro (robot description, xacro)
@@ -71,9 +71,10 @@
   <!-- laser — LiDAR scan frame                                           -->
   <!-- YDLIDAR typical: zero-angle points forward (+X), CCW rotation      -->
+  <!-- 8-29: 雷达 0° 标记实际朝车尾(装反 180°)，软件补偿 yaw=π            -->
   <!-- ================================================================= -->
   <joint name="laser_joint" type="fixed">
     <parent link="base_lidar_link"/>
     <child link="laser"/>
-    <origin xyz="0 0 0.03" rpy="0 0 0"/>
+    <origin xyz="0 0 0.03" rpy="0 0 3.14159"/>
   </joint>
   <link name="laser">

Commit message: fix: 撤销误判的雷达 180° 补偿（实测车头指示反向，雷达未装反）

File: ros2_ws/src/armbot_description/urdf/armbot.urdf.xacro (robot description, xacro)
@@ -71,10 +71,10 @@
   <!-- laser — LiDAR scan frame                                           -->
   <!-- YDLIDAR typical: zero-angle points forward (+X), CCW rotation      -->
-  <!-- 8-29: 雷达 0° 标记实际朝车尾(装反 180°)，软件补偿 yaw=π            -->
+  <!-- 8-29: 曾误判雷达装反 180° 加 yaw=π 补偿，实测车头指示反向，撤销恢复 0 -->
   <!-- ================================================================= -->
   <joint name="laser_joint" type="fixed">
     <parent link="base_lidar_link"/>
     <child link="laser"/>
-    <origin xyz="0 0 0.03" rpy="0 0 3.14159"/>
+    <origin xyz="0 0 0.03" rpy="0 0 0"/>
   </joint>
   <link name="laser">
